File: szendvicspanel/szendvicspanel/controller.kicad_sch (KiCad schematic)
At the start: 0 parts

Commit message: ANALOG_IN a mikrokontrolleres modulra is
Changed lines of the file:
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@@
+		)
+	)
+	(hierarchical_label "ANALOG_IN"
+		(shape input)
+		(at 52.07 71.12 0)
+		(effects
+			(font
+				(size 1.27 1.27)
+			)
+			(justify left)
 		)
 	)
 	(hierarchical_label "+5V"
 		(shape input)
-		(at 52.07 68.58 0)
+		(at 52.07 67.31 0)
 		(effects
 			(font
