File: szendvicspanel/szendvicspanel/jelgen.kicad_sch (KiCad schematic)
At the start: 0 parts

Commit message: V1
Parts:
- added C1: 3,2n, symbol Device:C
- added C2: 100n, symbol Device:C
- added J1: Conn_01x04_Pin, Connector_PinHeader_2.54mm:PinHeader_1x04_P2.54mm_Horizontal, symbol Connector:Conn_01x04_Pin
- added OJ1, OJ2, OJ3, OJ4, OJ5, OJ6, OJ7, OJ8: Conn_01x03_Socket, Connector_PinSocket_2.54mm:PinSocket_1x03_P2.54mm_Vertical, symbol Connector:Conn_01x03_Socket
- added R1, R4: 1k, symbol Device:R
- added R2: 2k, symbol Device:R
- added R3: 2,4k, symbol Device:R
- added RV1, RV2, RV4: R_Potentiometer, symbol Device:R_Potentiometer
- added TP1, TP2, TP3, TP4: TestPoint, Connector_PinHeader_2.54mm:PinHeader_1x01_P2.54mm_Vertical, symbol Connector:TestPoint
- added U1, U2: TL072, symbol Amplifier_Operational:TL072
Connections:
- net ANALOG_IN: now also C2.1, J1.2 (Pin_2)
- net GND: now also J1.1 (Pin_1), OJ1.2 (Pin_2), OJ2.2 (Pin_2), OJ3.2 (Pin_2), OJ4.2 (Pin_2), OJ5.2 (Pin_2), OJ6.2 (Pin_2), OJ7.2 (Pin_2), OJ8.2 (Pin_2), RV1.3, RV4.3
- net PWM: now also OJ1.3 (Pin_3), OJ2.3 (Pin_3), OJ3.3 (Pin_3), OJ4.3 (Pin_3), OJ5.3 (Pin_3), OJ6.3 (Pin_3), OJ7.3 (Pin_3), OJ8.3 (Pin_3), RV4.2, TP3.1
- net VPWR: now also J1.4 (Pin_4), OJ1.1 (Pin_1), OJ2.1 (Pin_1), OJ3.1 (Pin_1), OJ4.1 (Pin_1), OJ5.1 (Pin_1), OJ6.1 (Pin_1), OJ7.1 (Pin_1), OJ8.1 (Pin_1)
- new net: R1.2, R2.1, U1.5 (+)
- new net: RV1.2, U2.3 (+)
- new net: C2.2, R4.2, U2.5 (+)
- new net: C1.2, R3.2, U1.2 (-)
- new net: RV4.1, U2.7
- new net: R3.1, RV2.2
- new net REF: R4.1, TP4.1, U1.3 (+), U1.6 (-), U2.1, U2.2 (-)
- new net SQUARE: R2.2, RV2.1, TP1.1, U1.7
- new net TRIANGLE: C1.1, R1.1, TP2.1, U1.1, U2.6 (-)
- new net VPP: RV1.1
- no-connect marks 0 -> 2
Other:
- note added: "8 db PWM output, 8 db H-hídhoz"
- note added: "Analóg jelgenerátor"
- note added: "Input és tesztpontnak szolgáló output"
- note removed: "TODO: jelgenerátor + analóg modul"

Commit message: Update jelgen.kicad_sch
Connections:
- net SQUARE: no longer R2.2, RV2.1, U1.7
- net TRIANGLE renamed TRI
- new net SQR: R2.2, RV2.1, U1.7
Changed lines of the file:
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@@
+	)
+	(junction
+		(at 133.35 67.31)
+		(diameter 0)
+		(color 0 0 0 0)
 	)
 	(junction
@@
 	)
 	(junction
+		(at 50.8 45.72)
+		(diameter 0)
+		(color 0 0 0 0)
+	)
+	(junction
 		(at 104.14 46.99)
 		(diameter 0)
@@
 	(junction
 		(at 133.35 44.45)
+		(diameter 0)
+		(color 0 0 0 0)
+	)
+	(junction
+		(at 50.8 33.02)
 		(diameter 0)
 		(color 0 0 0 0)
@@
 	(wire
 		(pts
-			(xy 180.34 46.99) (xy 199.39 46.99)
-		)
-		(stroke
-			(width 0)
-			(type default)
-		)
-	)
-	(wire
-		(pts
 			(xy 214.63 125.73) (xy 189.23 125.73)
 		)
@@
 	(wire
 		(pts
+			(xy 46.99 45.72) (xy 50.8 45.72)
+		)
+		(stroke
+			(width 0)
+			(type default)
+		)
+	)
+	(wire
+		(pts
 			(xy 186.69 110.49) (xy 181.61 110.49)
 		)
@@
 	(wire
 		(pts
+			(xy 50.8 29.21) (xy 50.8 33.02)
+		)
+		(stroke
+			(width 0)
+			(type default)
+		)
+	)
+	(wire
+		(pts
+			(xy 71.12 82.55) (xy 76.2 82.55)
+		)
+		(stroke
+			(width 0)
+			(type default)
+		)
+	)
+	(wire
+		(pts
 			(xy 246.38 107.95) (xy 246.38 123.19)
 		)
@@
 	(wire
 		(pts
+			(xy 50.8 46.99) (xy 50.8 45.72)
+		)
+		(stroke
+			(width 0)
+			(type default)
+		)
+	)
+	(wire
+		(pts
+			(xy 46.99 33.02) (xy 50.8 33.02)
+		)
+		(stroke
+			(width 0)
+			(type default)
+		)
+	)
+	(wire
+		(pts
 			(xy 36.83 153.67) (xy 34.29 153.67)
 		)
@@
 	(wire
 		(pts
+			(xy 50.8 45.72) (xy 50.8 43.18)
+		)
+		(stroke
+			(width 0)
+			(type default)
+		)
+	)
+	(wire
+		(pts
 			(xy 254 125.73) (xy 248.92 125.73)
 		)
@@
 	(wire
 		(pts
-			(xy 66.04 82.55) (xy 76.2 82.55)
-		)
-		(stroke
-			(width 0)
-			(type default)
-		)
-	)
-	(wire
-		(pts
 			(xy 133.35 44.45) (xy 143.51 44.45)
 		)
@@
 	(wire
 		(pts
+			(xy 180.34 46.99) (xy 184.15 46.99)
+		)
+		(stroke
+			(width 0)
+			(type default)
+		)
+	)
+	(wire
+		(pts
 			(xy 96.52 67.31) (xy 96.52 87.63)
 		)
@@
 	(wire
 		(pts
+			(xy 133.35 67.31) (xy 135.89 67.31)
+		)
+		(stroke
+			(width 0)
+			(type default)
+		)
+	)
+	(wire
+		(pts
 			(xy 191.77 138.43) (xy 191.77 123.19)
 		)
@@
 		(pts
 			(xy 226.06 138.43) (xy 224.79 138.43)
+		)
+		(stroke
+			(width 0)
+			(type default)
+		)
+	)
+	(wire
+		(pts
+			(xy 50.8 33.02) (xy 50.8 35.56)
 		)
 		(stroke
@@
 	)
 	(label "TRIANGLE"
-		(at 99.06 90.17 180)
+		(at 96.52 87.63 180)
 		(effects
 			(font
@@
 		)
 	)
-	(label "SQUARE"
-		(at 199.39 46.99 0)
-		(effects
-			(font
-				(size 1.27 1.27)
-			)
-			(justify left bottom)
-		)
-	)
 	(label "REF"
 		(at 90.17 41.91 180)
@@
 		)
 	)
-	(label "ANALOG_IN"
-		(at 66.04 82.55 180)
-		(effects
-			(font
-				(size 1.27 1.27)
-			)
-			(justify right bottom)
-		)
-	)
 	(label "TRIANGLE"
 		(at 133.35 44.45 180)
@@
 			)
 			(justify left bottom)
+		)
+	)
+	(global_label "REF"
+		(shape input)
+		(at 100.33 49.53 0)
+		(fields_autoplaced yes)
+		(effects
+			(font
+				(size 1.27 1.27)
+			)
+			(justify left)
+		)
+		(property "Intersheetrefs" "${INTERSHEET_REFS}"
+			(at 106.8228 49.53 0)
+			(effects
+				(font
+					(size 1.27 1.27)
+				)
+				(justify left)
+				(hide yes)
+			)
+		)
+	)
+	(hierarchical_label "GND"
+		(shape input)
+		(at 46.99 45.72 180)
+		(effects
+			(font
+				(size 1.27 1.27)
+			)
+			(justify right)
+		)
+	)
+	(hierarchical_label "TRI"
+		(shape output)
+		(at 135.89 67.31 0)
+		(effects
+			(font
+				(size 1.27 1.27)
+			)
+			(justify left)
+		)
+	)
+	(hierarchical_label "SQR"
+		(shape output)
+		(at 184.15 46.99 0)
+		(effects
+			(font
+				(size 1.27 1.27)
+			)
+			(justify left)
 		)
 	)
@@
 			)
 			(justify left)
+		)
+	)
+	(hierarchical_label "VPP"
+		(shape input)
+		(at 46.99 33.02 180)
+		(effects
+			(font
+				(size 1.27 1.27)
+			)
+			(justify right)
+		)
+	)
+	(hierarchical_label "ANALOG_IN"
+		(shape input)
+		(at 71.12 82.55 180)
+		(effects
+			(font
+				(size 1.27 1.27)
+			)
+			(justify right)
 		)
 	)
@@
 	(symbol
 		(lib_id "power:GND")
-		(at 50.8 43.18 0)
+		(at 50.8 46.99 0)
 		(unit 1)
 		(exclude_from_sim no)
@@
 		(fields_autoplaced yes)
 		(property "Reference" "#PWR09"
-			(at 50.8 49.53 0)
+			(at 50.8 53.34 0)
 			(effects
 				(font
@@
 		)
 		(property "Value" "GND"
-			(at 50.8 48.26 0)
+			(at 50.8 52.07 0)
 			(effects
 				(font
@@
 		)
 		(property "Footprint" ""
-			(at 50.8 43.18 0)
+			(at 50.8 46.99 0)
 			(effects
 				(font
@@
 		)
 		(property "Datasheet" ""
-			(at 50.8 43.18 0)
+			(at 50.8 46.99 0)
 			(effects
 				(font
@@
 		)
 		(property "Description" "Power symbol creates a global label with name \"GND\" , ground"
-			(at 50.8 43.18 0)
+			(at 50.8 46.99 0)
 			(effects
 				(font
@@
 	(symbol
 		(lib_id "power:VPP")
-		(at 50.8 35.56 0)
+		(at 50.8 29.21 0)
 		(unit 1)
 		(exclude_from_sim no)
@@
 		(fields_autoplaced yes)
 		(property "Reference" "#PWR011"
-			(at 50.8 39.37 0)
+			(at 50.8 33.02 0)
 			(effects
 				(font
@@
 		)
 		(property "Value" "VPP"
-			(at 50.8 30.48 0)
+			(at 50.8 24.13 0)
 			(effects
 				(font
@@
 		)
 		(property "Footprint" ""
-			(at 50.8 35.56 0)
+			(at 50.8 29.21 0)
 			(effects
 				(font
@@
 		)
 		(property "Datasheet" ""
-			(at 50.8 35.56 0)
+			(at 50.8 29.21 0)
 			(effects
 				(font
@@
 		)
 		(property "Description" "Power symbol creates a global label with name \"VPP\""
-			(at 50.8 35.56 0)
-			(effects
-				(font
+			(at 50.8 29.21 0)
+			(effects
+				(font
