File: szendvicspanel/szendvicspanel/jelgen.kicad_sch (KiCad schematic)
At the start: 24 parts, among them J1 Conn_01x04_Pin, U1 TL072, U2 TL072

Commit message: Analóg jelgen schematic copy+paste, output busz, analóg interfész pinjeinek frissítése
Parts:
- removed C2: 100n, symbol Device:C
- removed R1, R4: 1k, symbol Device:R
- removed R2: 2k, symbol Device:R
- removed R3: 2,4k, symbol Device:R
- removed RV4: R_Potentiometer, symbol Device:R_Potentiometer
- added C3: 3,2n, Capacitor_THT:C_Axial_L5.1mm_D3.1mm_P7.50mm_Horizontal, symbol Device:C
- added R5, R7: 1k, Resistor_THT:R_Axial_DIN0204_L3.6mm_D1.6mm_P5.08mm_Horizontal, symbol Device:R
- added R6: 2,4k, Resistor_THT:R_Axial_DIN0204_L3.6mm_D1.6mm_P5.08mm_Horizontal, symbol Device:R
- added R8: 2k, Resistor_THT:R_Axial_DIN0204_L3.6mm_D1.6mm_P5.08mm_Horizontal, symbol Device:R
- added RV3: R_Potentiometer, Potentiometer_THT:Potentiometer_Bourns_3266Y_Vertical, symbol Device:R_Potentiometer
- added unit 3 of U1
- added unit 3 of U2
- C1: value 3,2n -> 100n; footprint (none) -> Capacitor_THT:C_Axial_L5.1mm_D3.1mm_P7.50mm_Horizontal
- RV1, RV2: footprint (none) -> Potentiometer_THT:Potentiometer_Bourns_3266Y_Vertical
- U1: footprint (none) -> Package_DIP:DIP-8_W7.62mm
- renumbered J1 to J3, OJ5 to OJ2, OJ2 to OJ3, OJ6 to OJ4, OJ3 to OJ5, OJ7 to OJ6, OJ4 to OJ7
Connections:
- net VPP is gone; now on net VPWR: RV1.1
- net ANALOG_IN: now also C1.1
- net GND: now also RV2.3, U1.4 (V-), U2.4 (V-)
- net PWM: now also RV2.2
- net REF: now also R5.2
- net SQUARE: now also R8.2, RV3.1; no longer RV2.1
- net TRIANGLE: now also C3.2, R7.1; no longer C1.1
- net VPWR: now also U1.8 (V+), U2.8 (V+)
- net at U1.5 (+): now also R7.2, R8.1
- net at U2.5 (+): now also C1.2, R5.1
- net at U1.2 (-): now also C3.1, R6.2; no longer C1.2
- net at U2.7: now also RV2.1
- net +5V: now reaches J3.3 (Pin_3)
- new net: R6.1, RV3.2
- no-connect marks 2 -> 3
Other:
- note added: "Az oszcillátor háromszögjeléből és az analóg bemenetből előállítja a PWM jelet"
- note added: "Előállít egy asszimetrikus négyszög- és háromszögjelet a REF feszültség körül, 2V és V_{PWR}-2V között"
- note added: "Előállítja a REF feszültséget a potméter értéke alapján"
- note added: "GND ANALOG_IN +5V VPWR"
- note added: "Kell az +5V input a mikrovezérlős modulnak, de itt nem használjuk fel."
- note added: "Oszcillátor"
- note removed: "Analóg jelgenerátor"
- title: (none) -> Jelgenerátor
- moved on the sheet: J3, OJ1, OJ2, OJ3, OJ4, OJ5, OJ6, OJ7, OJ8, TP1, TP2, TP3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
