File: szendvicspanel/H-híd/H-híd.kicad_pcb (KiCad board)
At the start: 2 copper layers, 29.5 x 39 mm, 12 parts, among them J1 Conn_01x03_Pin, J2 Conn_01x02_Socket

Commit message: takartás
Parts:
- R1, R2: renamed from 3k3; footprint Resistor_THT:R_Axial_DIN0207_L6.3mm_D2.5mm_P15.24mm_Horizontal -> Resistor_THT:R_Axial_DIN0309_L9.0mm_D3.2mm_P12.70mm_Horizontal
- R3, R4: renamed from 240; footprint Resistor_THT:R_Axial_DIN0207_L6.3mm_D2.5mm_P15.24mm_Horizontal -> Resistor_THT:R_Axial_DIN0309_L9.0mm_D3.2mm_P12.70mm_Horizontal
- renumbered BS170 to Q1, BS170 to Q2, BS170 to Q3, BS170 to Q4, BS250 to Q5, BS250 to Q6
Routing:
- net GND: track 59.1 -> 0.81 mm
- net Net-(Q3-G): track 13.1 -> 18.4 mm
- net Net-(Q2-D): track 21.1 -> 20.0 mm
- net Net-(Q1-D): track 29.9 -> 30.8 mm
- net /VPWR: track 84.1 -> 83.4 mm
- net Net-(Q4-G): track 17.7 -> 17.0 mm
- net (no net): vias 0 -> 1
- removed copper zone on F.Cu, net GND
