File: szendvicspanel/H-híd/H-híd.kicad_pcb (KiCad board)
At the start: 2 copper layers, 28.3 x 39 mm, 12 parts, among them J1 Conn_01x03_Pin, J2 Conn_01x02_Socket, Q1 BS170, Q2 BS170, Q3 BS170, Q4 BS170, Q5 BS250, Q6 BS250

Commit message: Megváltoztattam a min csíkszélességet és így már gyártható:-)
Parts:
- R1, R2, R3, R4: footprint Resistor_THT:R_Axial_DIN0309_L9.0mm_D3.2mm_P12.70mm_Horizontal -> Resistor_SMD:R_1210_3225Metric_Pad1.30x2.65mm_HandSolder; moved to B.Cu
- moved R2 142.1 mm to (99.8, 75.8), turned to 180 degrees
- moved R4 126.5 mm to (102.7, 88.0), turned to 0 degrees
- moved Q6 122.5 mm to (110.5, 84.8), turned to 90 degrees
- moved Q2 122.0 mm to (111.6, 99.7), turned to 0 degrees
- moved R3 114.4 mm to (105.7, 103.2), turned to 180 degrees
- moved J2 112.5 mm to (115.7, 73.0)
- moved Q4 112.1 mm to (121.8, 80.5)
- moved J1 111.1 mm to (117.9, 106.2)
- moved Q5 109.7 mm to (104.9, 80.6), turned to 180 degrees
- moved Q1 107.8 mm to (120.7, 91.6), turned to 180 degrees
- moved Q3 107.0 mm to (114.6, 79.2)
- moved R1 96.9 mm to (120.3, 100.2)
Routing:
- net /VPWR: track 84.3 -> 0.00 mm
- net Net-(Q1-D): track 31.5 -> 0.00 mm
- net Net-(Q3-G): track 18.4 -> 0.00 mm
- net Net-(Q2-D): track 17.4 -> 0.00 mm
- net Net-(Q4-G): track 17.0 -> 0.00 mm
- net /OUT_A: track 16.7 -> 0.00 mm
- net /OUT_B: track 14.7 -> 0.00 mm
- net /PWM: track 7.02 -> 0.00 mm
- removed copper zone on B.Cu, net GND
Other:
- board outline removed
