File: szendvicspanel/H-híd, panelizált/H-híd, panelizált.kicad_pcb (KiCad board)
At the start: 2 copper layers, 130.8 x 85.8 mm, 96 parts, among them J1 Conn_01x03_Pin, J2 Conn_01x02_Socket, Q1 BS170, Q2 BS170, Q3 BS170, Q4 BS170, Q5 BS250, Q6 BS250

Commit message: Megváltoztattam a min csíkszélességet és így már gyártható:-)
Parts:
- removed the J1 at (106.5, 82.5)
- removed the J1 at (173.9, 82.5)
- removed the J1 at (140.2, 127.4)
- removed the J1 at (140.2, 82.5)
- removed the J1 at (72.8, 127.4)
- removed the J1 at (106.5, 127.4)
- removed the J1 at (173.9, 127.4)
- removed the J2 at (105.3, 52.3)
- removed the J2 at (172.7, 52.3)
- removed the J2 at (139.0, 52.3)
- removed the J2 at (172.7, 97.2)
- removed the J2 at (105.3, 97.2)
- removed the J2 at (139.0, 97.2)
- removed the J2 at (71.6, 97.2)
- removed the Q1 at (71.2, 120.3)
- removed the Q1 at (138.6, 120.3)
- removed the Q1 at (172.2, 75.4)
- removed the Q1 at (138.6, 75.4)
- removed the Q1 at (104.8, 75.4)
- removed the Q1 at (104.8, 120.3)
- removed the Q1 at (172.2, 120.3)
- removed the Q2 at (178.6, 75.4)
- removed the Q2 at (144.9, 120.3)
- removed the Q2 at (144.9, 75.4)
- removed the Q2 at (111.2, 120.3)
- removed the Q2 at (77.5, 120.3)
- removed the Q2 at (111.2, 75.4)
- removed the Q2 at (178.6, 120.3)
- removed the Q3 at (98.2, 106.3)
- removed the Q3 at (131.9, 106.3)
- removed the Q3 at (64.5, 106.3)
- removed the Q3 at (98.2, 61.4)
- removed the Q3 at (165.6, 61.4)
- removed the Q3 at (165.6, 106.3)
- removed the Q3 at (131.9, 61.4)
- removed the Q4 at (144.9, 102.5)
- removed the Q4 at (111.2, 57.7)
- removed the Q4 at (178.6, 57.7)
- removed the Q4 at (111.2, 102.5)
- removed the Q4 at (77.5, 102.5)
- removed the Q4 at (144.9, 57.7)
- removed the Q4 at (178.6, 102.5)
- removed the Q5 at (158.8, 106.3)
- removed the Q5 at (91.4, 106.3)
- removed the Q5 at (57.7, 106.3)
- removed the Q5 at (91.4, 61.4)
- removed the Q5 at (158.8, 61.4)
- removed the Q5 at (125.1, 106.3)
- removed the Q5 at (125.1, 61.4)
- removed the Q6 at (111.2, 96.3)
- removed the Q6 at (178.6, 51.4)
- removed the Q6 at (77.5, 96.3)
- removed the Q6 at (144.9, 96.3)
- removed the Q6 at (111.2, 51.4)
- removed the Q6 at (178.6, 96.3)
- removed the Q6 at (144.9, 51.4)
- removed the R1 at (160.7, 128.4)
- removed the R1 at (160.7, 83.6)
- removed the R1 at (93.3, 83.6)
- removed the R1 at (93.3, 128.4)
- removed the R1 at (127.0, 83.6)
- removed the R1 at (127.0, 128.4)
- removed the R1 at (59.6, 128.4)
- removed the R2 at (81.0, 123.2)
- removed the R2 at (148.4, 78.4)
- removed the R2 at (148.4, 123.2)
- removed the R2 at (182.1, 78.4)
- removed the R2 at (114.7, 78.4)
- removed the R2 at (182.1, 123.2)
- removed the R2 at (114.7, 123.2)
- removed the R3 at (63.8, 125.7)
- removed the R3 at (131.2, 125.7)
- removed the R3 at (164.9, 125.7)
- removed the R3 at (131.2, 80.8)
- removed the R3 at (97.5, 125.7)
- removed the R3 at (164.9, 80.8)
- removed the R3 at (97.5, 80.8)
- removed the R4 at (105.7, 116.9)
- removed the R4 at (72.0, 116.9)
- removed the R4 at (173.1, 116.9)
- removed the R4 at (139.4, 116.9)
- removed the R4 at (139.4, 72.0)
- removed the R4 at (105.7, 72.0)
- removed the R4 at (173.1, 72.0)
- added J10: Conn_01x02_Socket, Connector_PinSocket_2.54mm:PinSocket_1x02_P2.54mm_Horizontal, F.Cu at (112.7, 104.1)
- added J11: Conn_01x03_Pin, Connector_PinHeader_2.54mm:PinHeader_1x03_P2.54mm_Horizontal, F.Cu at (154.2, 134.3)
- added J12: Conn_01x02_Socket, Connector_PinSocket_2.54mm:PinSocket_1x02_P2.54mm_Horizontal, F.Cu at (153.0, 104.1)
- added J3: Conn_01x03_Pin, Connector_PinHeader_2.54mm:PinHeader_1x03_P2.54mm_Horizontal, F.Cu at (113.9, 83.9)
- added J4: Conn_01x02_Socket, Connector_PinSocket_2.54mm:PinSocket_1x02_P2.54mm_Horizontal, F.Cu at (112.7, 53.7)
- added J5: Conn_01x03_Pin, Connector_PinHeader_2.54mm:PinHeader_1x03_P2.54mm_Horizontal, F.Cu at (154.2, 83.9)
- added J6: Conn_01x02_Socket, Connector_PinSocket_2.54mm:PinSocket_1x02_P2.54mm_Horizontal, F.Cu at (153.0, 53.7)
- added J7: Conn_01x03_Pin, Connector_PinHeader_2.54mm:PinHeader_1x03_P2.54mm_Horizontal, F.Cu at (194.5, 83.9)
- added J8: Conn_01x02_Socket, Connector_PinSocket_2.54mm:PinSocket_1x02_P2.54mm_Horizontal, F.Cu at (193.3, 53.7)
- added J9: Conn_01x03_Pin, Connector_PinHeader_2.54mm:PinHeader_1x03_P2.54mm_Horizontal, F.Cu at (113.9, 134.3)
- added Q10: BS170, Package_TO_SOT_THT:TO-92_Inline, F.Cu at (118.6, 60.0)
- added Q11: BS250, Package_TO_SOT_THT:TO-92_Inline, F.Cu at (98.8, 62.8)
- added Q12: BS250, Package_TO_SOT_THT:TO-92_Inline, F.Cu at (118.6, 52.4)
- added Q13: BS170, Package_TO_SOT_THT:TO-92_Inline, F.Cu at (152.6, 76.8)
- added Q14: BS170, Package_TO_SOT_THT:TO-92_Inline, F.Cu at (158.9, 76.8)
- added Q15: BS170, Package_TO_SOT_THT:TO-92_Inline, F.Cu at (146.7, 62.7)
- added Q16: BS170, Package_TO_SOT_THT:TO-92_Inline, F.Cu at (158.9, 60.0)
- added Q17: BS250, Package_TO_SOT_THT:TO-92_Inline, F.Cu at (139.1, 62.8)
- added Q18: BS250, Package_TO_SOT_THT:TO-92_Inline, F.Cu at (158.9, 52.4)
- added Q19: BS170, Package_TO_SOT_THT:TO-92_Inline, F.Cu at (192.9, 76.8)
- added Q20: BS170, Package_TO_SOT_THT:TO-92_Inline, F.Cu at (199.2, 76.8)
- added Q21: BS170, Package_TO_SOT_THT:TO-92_Inline, F.Cu at (187.0, 62.7)
- added Q22: BS170, Package_TO_SOT_THT:TO-92_Inline, F.Cu at (199.2, 60.0)
- added Q23: BS250, Package_TO_SOT_THT:TO-92_Inline, F.Cu at (179.4, 62.8)
- added Q24: BS250, Package_TO_SOT_THT:TO-92_Inline, F.Cu at (199.2, 52.4)
- added Q25: BS170, Package_TO_SOT_THT:TO-92_Inline, F.Cu at (112.3, 127.2)
- added Q26: BS170, Package_TO_SOT_THT:TO-92_Inline, F.Cu at (118.6, 127.2)
- added Q27: BS170, Package_TO_SOT_THT:TO-92_Inline, F.Cu at (106.4, 113.1)
- added Q28: BS170, Package_TO_SOT_THT:TO-92_Inline, F.Cu at (118.6, 110.4)
- added Q29: BS250, Package_TO_SOT_THT:TO-92_Inline, F.Cu at (98.8, 113.2)
- added Q30: BS250, Package_TO_SOT_THT:TO-92_Inline, F.Cu at (118.6, 102.8)
- added Q31: BS170, Package_TO_SOT_THT:TO-92_Inline, F.Cu at (152.6, 127.2)
- added Q32: BS170, Package_TO_SOT_THT:TO-92_Inline, F.Cu at (158.9, 127.2)
- added Q33: BS170, Package_TO_SOT_THT:TO-92_Inline, F.Cu at (146.7, 113.1)
- added Q34: BS170, Package_TO_SOT_THT:TO-92_Inline, F.Cu at (158.9, 110.4)
- added Q35: BS250, Package_TO_SOT_THT:TO-92_Inline, F.Cu at (139.1, 113.2)
- added Q36: BS250, Package_TO_SOT_THT:TO-92_Inline, F.Cu at (158.9, 102.8)
- added Q7: BS170, Package_TO_SOT_THT:TO-92_Inline, F.Cu at (112.3, 76.8)
- added Q8: BS170, Package_TO_SOT_THT:TO-92_Inline, F.Cu at (118.6, 76.8)
- added Q9: BS170, Package_TO_SOT_THT:TO-92_Inline, F.Cu at (106.4, 62.7)
- added R10: 3k3, Resistor_THT:R_Axial_DIN0309_L9.0mm_D3.2mm_P12.70mm_Horizontal, F.Cu at (162.4, 79.8)
- added R11: 240, Resistor_THT:R_Axial_DIN0309_L9.0mm_D3.2mm_P12.70mm_Horizontal, F.Cu at (145.2, 82.2)
- added R12: 240, Resistor_THT:R_Axial_DIN0309_L9.0mm_D3.2mm_P12.70mm_Horizontal, F.Cu at (153.4, 72.7)
- added R13: 3k3, Resistor_THT:R_Axial_DIN0309_L9.0mm_D3.2mm_P12.70mm_Horizontal, F.Cu at (181.3, 85.0)
- added R14: 3k3, Resistor_THT:R_Axial_DIN0309_L9.0mm_D3.2mm_P12.70mm_Horizontal, F.Cu at (202.7, 79.8)
- added R15: 240, Resistor_THT:R_Axial_DIN0309_L9.0mm_D3.2mm_P12.70mm_Horizontal, F.Cu at (185.5, 82.2)
- added R16: 240, Resistor_THT:R_Axial_DIN0309_L9.0mm_D3.2mm_P12.70mm_Horizontal, F.Cu at (193.7, 72.7)
- added R17: 3k3, Resistor_THT:R_Axial_DIN0309_L9.0mm_D3.2mm_P12.70mm_Horizontal, F.Cu at (100.7, 135.4)
- added R18: 3k3, Resistor_THT:R_Axial_DIN0309_L9.0mm_D3.2mm_P12.70mm_Horizontal, F.Cu at (122.1, 130.2)
- added R19: 240, Resistor_THT:R_Axial_DIN0309_L9.0mm_D3.2mm_P12.70mm_Horizontal, F.Cu at (104.9, 132.6)
- added R20: 240, Resistor_THT:R_Axial_DIN0309_L9.0mm_D3.2mm_P12.70mm_Horizontal, F.Cu at (113.1, 123.1)
- added R21: 3k3, Resistor_THT:R_Axial_DIN0309_L9.0mm_D3.2mm_P12.70mm_Horizontal, F.Cu at (141.0, 135.4)
- added R22: 3k3, Resistor_THT:R_Axial_DIN0309_L9.0mm_D3.2mm_P12.70mm_Horizontal, F.Cu at (162.4, 130.2)
- added R23: 240, Resistor_THT:R_Axial_DIN0309_L9.0mm_D3.2mm_P12.70mm_Horizontal, F.Cu at (145.2, 132.6)
- added R24: 240, Resistor_THT:R_Axial_DIN0309_L9.0mm_D3.2mm_P12.70mm_Horizontal, F.Cu at (153.4, 123.1)
- added R5: 3k3, Resistor_THT:R_Axial_DIN0309_L9.0mm_D3.2mm_P12.70mm_Horizontal, F.Cu at (100.7, 85.0)
- added R6: 3k3, Resistor_THT:R_Axial_DIN0309_L9.0mm_D3.2mm_P12.70mm_Horizontal, F.Cu at (122.1, 79.8)
- added R7: 240, Resistor_THT:R_Axial_DIN0309_L9.0mm_D3.2mm_P12.70mm_Horizontal, F.Cu at (104.9, 82.2)
- added R8: 240, Resistor_THT:R_Axial_DIN0309_L9.0mm_D3.2mm_P12.70mm_Horizontal, F.Cu at (113.1, 72.7)
- added R9: 3k3, Resistor_THT:R_Axial_DIN0309_L9.0mm_D3.2mm_P12.70mm_Horizontal, F.Cu at (141.0, 85.0)
- moved Q3 133.0 mm to (187.0, 113.1)
- moved Q4 132.7 mm to (199.2, 110.4)
- moved J1 132.3 mm to (194.5, 134.3)
- moved J2 132.3 mm to (193.3, 104.1)
- moved Q1 132.3 mm to (192.9, 127.2)
- moved Q2 132.3 mm to (199.2, 127.2)
- moved Q5 132.3 mm to (179.4, 113.2)
- moved R1 132.3 mm to (181.3, 135.4)
- moved R2 132.3 mm to (202.7, 130.2)
- moved R3 132.3 mm to (185.5, 132.6)
- moved Q6 132.1 mm to (199.2, 102.8)
- moved R4 132.0 mm to (193.7, 123.1)
Routing:
- net /VPWR: track 674.5 -> 490.0 mm
- net Net-(Q1-D): track 251.9 -> 187.5 mm
- net Net-(Q3-G): track 147.4 -> 108.2 mm
- net Net-(Q2-D): track 139.1 -> 100.1 mm
- net /OUT_B: track 118.0 -> 82.7 mm
- net /OUT_A: track 133.3 -> 107.0 mm
- net Net-(Q4-G): track 135.6 -> 124.9 mm
- net /PWM: track 56.2 -> 57.4 mm
- net (no net): vias 1 -> 0
- added copper zone on F.Cu, net GND
Other:
- board size 130.8 x 85.8 mm -> 112.9 x 93.1 mm
